File: hardware/probe_b/probe_b.sch (KiCad schematic (older format))
At the start: 29 parts, among them J1 TEST_1P, J3 TEST_1P, J4 TEST_1P, J5 TEST_1P, J7 Conn_01x04, Q1 SI3415, U1 ATTINY25-20PU

Commit message: Probe B as Rev 1 as manufactured.
Parts:
- R1: value 10K -> 15K
- R7, R8: value R -> 1K
- R9: value 2K -> 1K
Connections:
- net labels added: Anode, Cathode
Other:
- note added: "Probe side shall have no pullup on I2C lines,\npullup must be enabled on master side only.\n\nAssuming pull up is around 20k and logic low \nthreshold of 2V (Vcc=5V) this gives R7 = R8 < 13.3k\n\nPicking R7=R8=1k limits current to 5 mA and then BAT54C-7-F \nhas Vf approx 360 mV which is within tolerance for negative \nvoltage on pins of ATtiny. While leaving maximal noise margin."
- note added: "Typical Vf of 2V for D1, then R9=1K \nwould result in 3 mA or around\n15% brightness for a If 20mA LED.\n"
Changed lines of the file:
@@
 P 750 3200
 F 0 "R1" V 830 3200 50  0000 C CNN
-F 1 "10K" V 750 3200 50  0000 C CNN
+F 1 "15K" V 750 3200 50  0000 C CNN
 F 2 "Resistors_SMD:R_0603" V 680 3200 50  0001 C CNN
 F 3 "" H 750 3200 50  0001 C CNN
@@
 P 7050 3300
 F 0 "R9" V 6950 3300 50  0000 C CNN
-F 1 "2K" V 7050 3300 50  0000 C CNN
+F 1 "1K" V 7050 3300 50  0000 C CNN
 F 2 "Resistors_SMD:R_0603" V 6980 3300 50  0001 C CNN
 F 3 "" H 7050 3300 50  0001 C CNN
@@
 P 4900 4550
 F 0 "R7" V 4800 4550 50  0000 C CNN
-F 1 "R" V 4900 4550 50  0000 C CNN
+F 1 "1K" V 4900 4550 50  0000 C CNN
 F 2 "Resistors_SMD:R_0603" V 4830 4550 50  0001 C CNN
 F 3 "" H 4900 4550 50  0001 C CNN
@@
 P 4900 4650
 F 0 "R8" V 4980 4650 50  0000 C CNN
-F 1 "R" V 4900 4650 50  0000 C CNN
+F 1 "1K" V 4900 4650 50  0000 C CNN
 F 2 "Resistors_SMD:R_0603" V 4830 4650 50  0001 C CNN
 F 3 "" H 4900 4650 50  0001 C CNN
@@
 Wire Wire Line
 	2400 1800 2200 1800
+Text Notes 3450 5850 0    39   ~ 0
+Probe side shall have no pullup on I2C lines,\npullup must be enabled on master side only.\n\nAssuming pull up is around 20k and logic low \nthreshold of 2V (Vcc=5V) this gives R7 = R8 < 13.3k\n\nPicking R7=R8=1k limits current to 5 mA and then BAT54C-7-F \nhas Vf approx 360 mV which is within tolerance for negative \nvoltage on pins of ATtiny. While leaving maximal noise margin.
+Text Notes 6700 3800 0    39   ~ 0
+Typical Vf of 2V for D1, then R9=1K \nwould result in 3 mA or around\n15% brightness for a If 20mA LED.\n
+Text Label 2300 1800 1    60   ~ 0
+Anode
+Text Label 2300 2050 0    60   ~ 0
+Cathode
 $EndSCHEMATC

Commit message: Fixes #21. Also removes RC filters that made the output impedence too high for the ADC. Changed connector to Micro USB due to cable availabiliy. Changed to a more reasonable inline ferrite and also removed ptc fuse due to too high Vdrop. Series resistors for I2C righ-sized.
Parts:
- removed C1, C2, C6, C7: 100nF, Capacitors_SMD:C_0603, symbol C
- removed F1: Polyfuse_Small, digikey-footprints:0603, symbol Polyfuse_Small
- removed J4, J5: TEST_1P, Measurement_Points:Measurement_Point_Round-SMD-Pad_Small, symbol TEST_1P
- removed J7: Conn_01x04, Connectors_JST:JST_EH_S04B-EH_04x2.50mm_Angled, symbol Conn_01x04
- removed R2, R3, R5, R6: 100K, Resistors_SMD:R_0603, symbol R
- added J2: USB_A, Connect:USB_Micro-B, symbol USB_A
- D1: value LED -> PWR_LED
- D2: value D_Zener -> BZT52C5V6
- D3: value BAT54C-7-F -> BAT54C
- L1: footprint digikey-footprints:Inductor_13R106C -> Inductors_THT:L_Axial_L5.3mm_D2.2mm_P7.62mm_Horizontal_Vishay_IM-1
- Q1: value SI3415 -> SI2323DS; footprint TO_SOT_Packages_SMD:SOT-23 -> emilibeda:SOT-23-Power
- R7, R8: value 1K -> 33R
Connections:
- wire segments 42 -> 31
- no-connect marks 0 -> 1
Other:
- note added: "BAT54C max avg 200mA @ 5 V -> 25 R series resistance.\nPick 33 R for some headroom (E6 value)."
- note added: "MCU max active current internal 8 Mhz osc. 5: 5 mA\nProbes are less than 1 mA together\nPower LED is 3 mA with listed parts\nI2C is bounded by 10 mA due to series resistors \nSum total: 19 mA"
- note added: "We send I2C over USB cables.\nUSB micro cables are easy to find and designed\nfor high speed data transfer and shielded. We can't\nfind a more apt and readily available cable."
- moved on the sheet: J1, NTC1, R1
