File: hardware/probe_b/probe_b.sch (KiCad schematic (older format))
At the start: 47 parts, among them J1 ICSP, J2 PUMP, J3 PUMP, J4 C_sense, J5 Daisy_OUT, J6 Daisy_IN, J7 TEMP_A, Q1 SI2323DS, U1 ATMEGA328P-AU, U2 MIC94090

Commit message: V3 of the node.G
Parts:
- D1, D3, D4: symbol dk_Diodes-Rectifiers-Arrays:BAT54S-7-F -> probe_b-rescue:BAT54S-7-F-dk_Diodes-Rectifiers-Arrays
- D6: symbol dk_Diodes-Rectifiers-Single:MBR0520LT1G -> probe_b-rescue:MBR0520LT1G-dk_Diodes-Rectifiers-Single
- U2: symbol mic94090:MIC94090 -> probe_b-rescue:MIC94090-mic94090
Changed lines of the file:
@@
 I2C Design\n* Standard Speed (100 KHz, 10 us period)\n* Rise/Fall time = 1 us\n* Given 200R input series resistance pullup must be [2K7, 4K5]\n   assuming max allowed 400 pF bus capacitance\n* Pull up only on pump side, not on probes\n* Total bus capacitance < 400 pFu
 $Comp
-L dk_Diodes-Rectifiers-Arrays:BAT54S-7-F D1
+L probe_b-rescue:BAT54S-7-F-dk_Diodes-Rectifiers-Arrays D1
 U 1 1 5B9DFD9E
 P 3650 1300
@@
 $EndComp
 $Comp
-L dk_Diodes-Rectifiers-Arrays:BAT54S-7-F D3
+L probe_b-rescue:BAT54S-7-F-dk_Diodes-Rectifiers-Arrays D3
 U 1 1 5B9E0005
 P 4050 1300
@@
 $EndComp
 $Comp
-L dk_Diodes-Rectifiers-Arrays:BAT54S-7-F D4
+L probe_b-rescue:BAT54S-7-F-dk_Diodes-Rectifiers-Arrays D4
 U 1 1 5B9E0534
 P 4500 2550
@@
 	2550 2500 2800 2500
 $Comp
-L mic94090:MIC94090 U2
+L probe_b-rescue:MIC94090-mic94090 U2
 U 1 1 5B9D4F60
 P 5250 5250
@@
 	6000 5000 6000 4900
 $Comp
-L dk_Diodes-Rectifiers-Single:MBR0520LT1G D6
+L probe_b-rescue:MBR0520LT1G-dk_Diodes-Rectifiers-Single D6
 U 1 1 5BA31025
 P 5750 4900
