File: hardware/node/node.kicad_pcb (KiCad board)
At the start: 2 copper layers, 135.9 x 25.4 mm, 48 parts, among them J1 IN, J10 ICSP, J30 PUMP, J60 OVF, Q0 SI2323DS, U1 ATmega328P-AU, U2 LMC555xM, U3 TPS22810, U4 P82B96

Commit message: Updating layout of node and art.
Parts:
- removed C20, C60: 100nF, Capacitor_SMD:C_0603_1608Metric_Pad1.05x0.95mm_HandSolder
- removed C21, C22: 10nF, Capacitor_SMD:C_0603_1608Metric_Pad1.05x0.95mm_HandSolder
- removed R10: 1K, Resistor_SMD:R_0603_1608Metric_Pad1.05x0.95mm_HandSolder
- removed R24: 0R, Resistor_SMD:R_0603_1608Metric_Pad1.05x0.95mm_HandSolder
- removed TP20: A, TestPoint:TestPoint_Pad_D1.0mm
- removed U2: LMC555xM, Package_SO:SOIC-8_3.9x4.9mm_P1.27mm
- added A0: ART, emilibeda:waterino_small_12_3mm, B.Cu at (-70.2, 59.0)
- added A1: ART, emilibeda:OSH_7_3mm, B.Cu at (-65.0, 11.8)
- added D11: D_RST, Diode_SMD:D_SOD-123, F.Cu at (-75.8, 47.5)
- C10, C30, C40: moved to B.Cu
- C12, C14: value 10nF -> 100nF
- R11, R61: value 51K -> 1K
- R20: value 125R -> 1K
- R21: value 1M -> 1K
- R22: value 100K -> 1K
- R23: value 10K -> 100K
- moved TH50 286.6 mm to (-70.0, 178.0), turned to 90 degrees
- moved J60 218.3 mm to (-63.5, 23.0), turned to 270 degrees
- moved F0 214.8 mm to (-77.5, 9.50)
- moved R11 214.2 mm to (-76.5, 49.5)
- moved R23 214.0 mm to (-67.5, 64.0)
- moved R61 212.3 mm to (-71.0, 48.0), turned to 90 degrees
- moved C50 211.8 mm to (-62.5, 52.0), turned to 90 degrees
- moved D0 210.8 mm to (-77.5, 14.5), turned to 270 degrees
- moved R60 209.7 mm to (-69.0, 48.0), turned to 90 degrees
- moved R51 209.5 mm to (-62.5, 56.5), turned to 270 degrees
- moved D30 208.9 mm to (-66.2, 37.2), turned to 90 degrees
- moved Q0 208.1 mm to (-76.5, 25.2)
- moved R50 207.3 mm to (-62.5, 61.0), turned to 90 degrees
- moved C12 206.1 mm to (-77.5, 60.0), turned to 180 degrees
- moved J1 206.1 mm to (-74.5, 15.0), turned to 90 degrees
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Connections:
- C14 pad 1: Vcc -> RST
- C50 pad 1: Net-(C50-Pad1) -> TEMP_SENSE
- J1 pad 2: Vin -> +12V
- J1 pad 6: +12V -> Vin
- R11 pad 1: Net-(R10-Pad2) -> Vcc
- R11 pad 2: GND -> RST
- R20 pad 1: F_PROBE_EN -> C_SENS_TOP
- R20 pad 2: Net-(C20-Pad1) -> C_SENS_REF
- R21 pad 1: Net-(C20-Pad1) -> C_SENS_REF
- R21 pad 2: Net-(C22-Pad1) -> Net-(R21-Pad2)
- R22 pad 1: F_PROBE -> Net-(R21-Pad2)
- R22 pad 2: Net-(C22-Pad1) -> C_SENS_BOT
- R23 pad 1: Net-(C22-Pad1) -> C_SENS_TOP
- R23 pad 2: /PROBE_K -> C_SENS_TRK
- R50 pad 2: Net-(C50-Pad1) -> Net-(R50-Pad2)
- R51 pad 2: Net-(C50-Pad1) -> Net-(R50-Pad2)
- TH50 pad 1: Net-(C50-Pad1) -> Net-(R50-Pad2)
- U1 pad 10: Net-(R10-Pad2) -> C_SENS_REF
- U1 pad 11: OVF_SENSE -> C_SENS_TRK
- U1 pad 12: OVF_EN -> Net-(U1-Pad12)
- U1 pad 13: LED_EN -> ~TEMP_EXC
- U1 pad 14: ~TEMP_EXC -> Net-(U1-Pad14)
- U1 pad 25: Net-(U1-Pad25) -> OVF_EN
- U1 pad 26: Net-(U1-Pad26) -> OVF_SENSE
- U1 pad 7: Net-(U1-Pad7) -> C_SENS_BOT
- U1 pad 8: F_PROBE_EN -> C_SENS_TOP
- U1 pad 9: F_PROBE -> LED_EN
Routing:
- net Net-(R50-Pad2): track 0.00 -> 127.6 mm
- net C_SENS_TRK: track 0.00 -> 115.3 mm
- net Net-(C50-Pad1): track 89.6 -> 0.00 mm
- net GND: track 37.6 -> 4.63 mm, vias 22 -> 99
- net +12V: track 16.6 -> 46.4 mm
- net Net-(C22-Pad1): track 23.0 -> 0.00 mm
- net /Pump+: track 34.7 -> 12.1 mm
- net SCK: track 7.02 -> 26.0 mm, vias 0 -> 2
- net Net-(J60-Pad1): track 10.9 -> 28.4 mm
- net Vin: track 28.0 -> 45.1 mm, vias 1 -> 0
- net /F_in: track 0.00 -> 15.4 mm
- net Net-(C20-Pad1): track 15.1 -> 0.00 mm
- net TEMP_SENSE: track 23.9 -> 9.28 mm, vias 2 -> 0
- net ~TEMP_EXC: track 111.6 -> 125.9 mm, vias 2 -> 0
- net MOSI: track 15.7 -> 29.6 mm, vias 0 -> 2
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- added copper zone on F.Cu, net GND
- removed copper zone on F.Cu, net /F_in
- removed copper zone on F.Cu, net /PROBE_A
- removed copper zone on B.Cu, net /PROBE_K
- removed copper zone on F.Cu, net /PROBE_K
Other:
- board size 135.9 x 25.4 mm -> 20 x 180 mm
- net class Default: clearance 0.22 -> 0.2; trace_width 0.22 -> 0.2; via_dia 0.44 -> 0.5
- rule trace_clearance: 0.22 -> 0.2
- rule trace_min: 0.22 -> 0.2
- rule via_min_size: 0.4 -> 0.45
- board text added: "SCL"
- board text added: "SDA"
- board text added: "SENS"
- board text added: "SENSE"
- board text added: "Soil up to HERE"
- board text added: "Waterino: Node Rev 1.0"
- board text removed: "0V"
- board text removed: "OVF+"
